File: schematic/petdisk.kicad_sch (KiCad schematic)
At the start: 15 parts, among them J1 IEEE-488-GPIB, J2 microSD, J3 PET-TAPE, U1 STM8S105K6T6C, U2 AMS1117-3.3

Commit message: fix: rewrite petdisk.kicad_sch to valid KiCad 7 format
- Add top-level uuid and lib_symbols section with symbol
  definitions for all 9 component types
- Fix global_label: add label text as first argument
- Replace net_label with label (text as first argument)
- Replace power_symbol with symbol (lib_id power:GND / power:+5V)
- Remove invalid (at ...) from pin instances inside symbols;
  only (uuid ...) is valid there per KiCad parser
- Add sheet_instances footer

Agent-Logs-Url: https://github.com/beroset/petdisk/sessions/8b06b753-060c-4b91-baf3-7e19dc0b9543

Co-authored-by: beroset <4911249+beroset@users.noreply.github.com>
Connections:
- new net: C4.1, U1.PA3
- new net +5V: U2.VIN
- new net ATN: J1.1
- new net DAV: J1.6, U1.PB1
- new net DIO1: J1.11, U1.PD1
- new net DIO2: J1.10, U1.PD0
- new net DIO3: J1.9
- new net DIO4: J1.8, U1.PB7
- new net DIO5: J1.23, U1.PB6
- new net DIO6: J1.22, U1.PB5
- new net DIO7: J1.21, U1.PB4
- new net DIO8: J1.20, U1.PB3
- new net EOI: J1.7
- new net GND: J1.13, J1.14, J1.15, J1.16, J1.17, J1.18, J2.3, J3.3, R2.2, R4.2, R6.2
- new net IFC: J1.3
- new net NDAC: J1.4
- new net NRFD: J1.5, U1.PB0
- new net PA3_NSS: R5.1
- new net PC5_SCK: R1.1
- new net PC6_MOSI: R3.1
- new net REN: J1.19
- new net SD_CS: J2.5, R5.2
- new net SD_MOSI: J2.4, R3.2
- new net SD_SCK: J2.1, R1.2
- new net SRQ: J1.2
- new net VCC_3V3: J2.2, U2.VOUT
